File: schematic/MyWallSwitch/MyWallSwitch.kicad_pcb (KiCad board)
At the start: 2 copper layers, 29.8 x 44.8 mm, 19 parts, among them J1 Screw_Terminal_01x04, J2 TTL, J3 AVR-ISP-6, SW1 SW_Push, U1 HLK-PM03 (3.3 1A), U2 ATmega328P-AU, U3 AQH3213, U4 NRF24L01, Y1 Resonator

Commit message: Fix Shematic and PCB
Parts:
- removed C5: 100n, Capacitors_SMD:C_0603_HandSoldering
- U3: footprint Housings_DIP:DIP-8_W7.62mm_SMDSocket_SmallPads -> ennys:AQH32xxA
- moved U3 6.02 mm to (144.9, 82.2), turned to 270 degrees
- moved C1 2.83 mm to (143.5, 105.0)
- moved U2 0.76 mm to (137.2, 108.5)
Connections:
- J3 pad 5: Net-(C5-Pad1) -> Net-(C4-Pad2)
- U2 pad 30: Net-(J2-Pad2) -> Net-(J2-Pad3)
- U2 pad 31: Net-(J2-Pad3) -> Net-(J2-Pad2)
- Y1 pad 2: (no net) -> GND
Routing:
- net GND: track 131.8 -> 151.8 mm, vias 0 -> 1
- net Net-(J2-Pad2): track 5.74 -> 25.1 mm, vias 0 -> 1
- net Net-(C4-Pad2): track 27.6 -> 42.9 mm, vias 0 -> 2
- net Net-(C5-Pad1): track 13.5 -> 0.00 mm, vias 2 -> 0
- net Net-(R1-Pad2): track 23.4 -> 18.3 mm, vias 2 -> 0
- net Net-(U2-Pad7): track 19.3 -> 23.9 mm
- net VCC: track 60.1 -> 56.8 mm, vias 1 -> 0
- net Net-(C1-Pad1): track 11.6 -> 12.8 mm
- net Net-(U2-Pad8): track 17.2 -> 18.0 mm
- net Net-(U2-Pad14): track 15.9 -> 15.1 mm
- net Net-(U2-Pad13): track 14.3 -> 13.5 mm
- net Net-(R1-Pad1): track 8.63 -> 7.87 mm
- net Net-(J3-Pad3): track 26.7 -> 27.5 mm
- net Net-(C3-Pad2): track 29.7 -> 30.3 mm
- net Net-(J2-Pad3): track 4.94 -> 5.52 mm
- added copper zone on B.Cu, net GND
- added copper zone on F.Cu, net GND
