File: schematic/MyWallSwitch/MyWallSwitch.sch (KiCad schematic (older format))
At the start: 20 parts, among them J1 Screw_Terminal_01x03, J2 TTL, J3 AVR-ISP-6, SW1 SW_Push, U1 HLK-PM03 (3.3 1A), U2 ATmega328P-AU, U3 AQH3213, U4 NRF24L01, Y1 Resonator

Commit message: firmware build
Parts:
- removed F2: 300mA slow, symbol Device:Fuse
- removed J1: Screw_Terminal_01x03, symbol Connector:Screw_Terminal_01x03
- added J1: Screw_Terminal_01x04, Connectors_Terminal_Blocks:TerminalBlock_bornier-4_P5.08mm, symbol Connector:Screw_Terminal_01x04
- C1, C2, C3, C4, C6: footprint (none) -> Capacitors_SMD:C_0603_HandSoldering
- C5: value C -> 100n; footprint (none) -> Capacitors_SMD:C_0603_HandSoldering
- F1: value 1.2 A -> BK/GMD-1.2R; footprint (none) -> Fuse_Holders_and_Fuses:Fuseholder5x20_horiz_SemiClosed_Casing10x25mm
- J2: footprint (none) -> Pin_Headers:Pin_Header_Straight_1x06_Pitch2.54mm
- J3: footprint (none) -> Pin_Headers:Pin_Header_Straight_2x03_Pitch2.54mm
- R1: value R -> 220R; footprint (none) -> Resistors_SMD:R_0603_HandSoldering
- R2: footprint (none) -> Resistors_SMD:R_0603_HandSoldering
- RV1: value Varistor -> MOV-07D391KTR; footprint (none) -> Varistors:RV_Disc_D7_W5.5_P5
- SW1: footprint (none) -> Buttons_Switches_SMD:SW_SPST_B3S-1000
- U1: footprint (none) -> ennys:HLK-PM01
- U2: footprint Package_QFP:TQFP-32_7x7mm_P0.8mm -> Housings_QFP:TQFP-32_7x7mm_Pitch0.8mm
- U3: footprint (none) -> Housings_DIP:DIP-8_W7.62mm_SMDSocket_SmallPads
- U4: footprint (none) -> mysensors_radios:NRF24L01-SMD
- Y1: footprint (none) -> ennys:Resonator_Ceramic
Connections:
- net L_OUT: now also J1.4 (Pin_4)
- net at RV1.1, U1.1 (AC(L)): now also F1.1, J1.1 (Pin_1)
- net at RV1.2, U1.2 (AC(L)): now also J1.2 (Pin_2), J1.3 (Pin_3)
Other:
- moved on the sheet: F1
Changed lines of the file:
@@
 EESchema Schematic File Version 4
+LIBS:MyWallSwitch-cache
 EELAYER 26 0
 EELAYER END
@@
 F 0 "U2" H 4500 2164 50  0000 C CNN
 F 1 "ATmega328P-AU" H 4500 2073 50  0000 C CNN
-F 2 "Package_QFP:TQFP-32_7x7mm_P0.8mm" H 4500 3750 50  0001 C CIN
+F 2 "Housings_QFP:TQFP-32_7x7mm_Pitch0.8mm" H 4500 3750 50  0001 C CIN
 F 3 "http://ww1.microchip.com/downloads/en/DeviceDoc/ATmega328_P%20AVR%20MCU%20with%20picoPower%20Technology%20Data%20Sheet%2040001984A.pdf" H 4500 3750 50  0001 C CNN
 	1    4500 3750
@@
 F 0 "Y1" V 5846 3311 50  0000 L CNN
 F 1 "Resonator" V 5755 3311 50  0000 L CNN
-F 2 "" H 5775 3200 50  0001 C CNN
+F 2 "ennys:Resonator_Ceramic" H 5775 3200 50  0001 C CNN
 F 3 "~" H 5775 3200 50  0001 C CNN
 	1    5800 3200
@@
 F 0 "U4" H 7600 3250 60  0000 C CNN
 F 1 "NRF24L01" H 7600 3144 60  0000 C CNN
-F 2 "" H 7600 2550 60  0000 C CNN
+F 2 "mysensors_radios:NRF24L01-SMD" H 7600 2550 60  0001 C CNN
 F 3 "" H 7600 2550 60  0000 C CNN
 	1    7600 2700
@@
 F 0 "U1" H 3100 2137 60  0000 C CNN
 F 1 "HLK-PM03 (3.3 1A)" H 3100 2031 60  0000 C CNN
-F 2 "" H 3100 1550 60  0001 C CNN
+F 2 "ennys:HLK-PM01" H 3100 1550 60  0001 C CNN
 F 3 "" H 3100 1550 60  0001 C CNN
 	1    3100 1550
 	1    0    0    -1
-$EndComp
-$Comp
-L Device:Fuse F2
-U 1 1 5C2D1BA7
-P 1800 1450
-F 0 "F2" V 1603 1450 50  0000 C CNN
-F 1 "300mA slow" V 1694 1450 50  0000 C CNN
-F 2 "" V 1730 1450 50  0001 C CNN
-F 3 "~" H 1800 1450 50  0001 C CNN
-	1    1800 1450
-	0    1    1    0
 $EndComp
 $Comp
@@
 P 2100 1600
 F 0 "RV1" H 2203 1646 50  0000 L CNN
-F 1 "Varistor" H 2203 1555 50  0000 L CNN
-F 2 "" V 2030 1600 50  0001 C CNN
+F 1 "MOV-07D391KTR" H 2203 1555 50  0000 L CNN
+F 2 "Varistors:RV_Disc_D7_W5.5_P5" V 2030 1600 50  0001 C CNN
 F 3 "~" H 2100 1600 50  0001 C CNN
 	1    2100 1600
@@
 	2550 1750 2550 1700
 Wire Wire Line
-	2100 1450 2550 1450
+	2100 1450 2150 1450
 Wire Wire Line
 	2550 1450 2550 1500
-$Comp
-L Connector:Screw_Terminal_01x03 J1
-U 1 1 5C2D1D9B
-P 1050 1550
-F 0 "J1" H 970 1225 50  0000 C CNN
-F 1 "Screw_Terminal_01x03" H 970 1316 50  0000 C CNN
-F 2 "" H 1050 1550 50  0001 C CNN
-F 3 "~" H 1050 1550 50  0001 C CNN
-	1    1050 1550
-	-1   0    0    1
-$EndComp
-Wire Wire Line
-	1950 1450 2100 1450
 Connection ~ 2100 1450
 Wire Wire Line
-	1250 1450 1550 1450
-Wire Wire Line
-	1250 1550 1800 1550
+	1250 1550 1300 1550
 Wire Wire Line
 	1800 1550 1800 1750
@@
 F 0 "C1" H 3465 2746 50  0000 L CNN
 F 1 "100n" H 3465 2655 50  0000 L CNN
-F 2 "" H 3388 2550 50  0001 C CNN
+F 2 "Capacitors_SMD:C_0603_HandSoldering" H 3388 2550 50  0001 C CNN
 F 3 "~" H 3350 2700 50  0001 C CNN
 	1    3350 2700
@@
 F 0 "C6" H 8265 2946 50  0000 L CNN
 F 1 "100n" H 8265 2855 50  0000 L CNN
-F 2 "" H 8188 2750 50  0001 C CNN
+F 2 "Capacitors_SMD:C_0603_HandSoldering" H 8188 2750 50  0001 C CNN
 F 3 "~" H 8150 2900 50  0001 C CNN
 	1    8150 2900
@@
 F 0 "J3" H 6620 3504 50  0000 R CNN
 F 1 "AVR-ISP-6" H 6620 3595 50  0000 R CNN
-F 2 "" V 6650 3550 50  0001 C CNN
+F 2 "Pin_Headers:Pin_Header_Straight_2x03_Pitch2.54mm" V 6650 3550 50  0001 C CNN
 F 3 " ~" H 5625 2950 50  0001 C CNN
 	1    6900 3500
@@
 F 0 "R2" V 5943 4050 50  0000 C CNN
 F 1 "10k" V 6034 4050 50  0000 C CNN
-F 2 "" V 6080 4050 50  0001 C CNN
+F 2 "Resistors_SMD:R_0603_HandSoldering" V 6080 4050 50  0001 C CNN
 F 3 "~" H 6150 4050 50  0001 C CNN
 	1    6150 4050
@@
 P 6200 3400
 F 0 "C5" V 5948 3400 50  0000 C CNN
-F 1 "C" V 6039 3400 50  0000 C CNN
-F 2 "" H 6238 3250 50  0001 C CNN
+F 1 "100n" V 6039 3400 50  0000 C CNN
+F 2 "Capacitors_SMD:C_0603_HandSoldering" H 6238 3250 50  0001 C CNN
 F 3 "~" H 6200 3400 50  0001 C CNN
 	1    6200 3400
@@
 F 0 "J2" H 6678 4426 50  0000 L CNN
 F 1 "TTL" H 6678 4335 50  0000 L CNN
-F 2 "" H 6650 4450 50  0001 C CNN
+F 2 "Pin_Headers:Pin_Header_Straight_1x06_Pitch2.54mm" H 6650 4450 50  0001 C CNN
 F 3 "~" H 6650 4450 50  0001 C CNN
 	1    6650 4450
@@
 F 0 "C4" V 5698 4250 50  0000 C CNN
 F 1 "100n" V 5789 4250 50  0000 C CNN
-F 2 "" H 5988 4100 50  0001 C CNN
+F 2 "Capacitors_SMD:C_0603_HandSoldering" H 5988 4100 50  0001 C CNN
 F 3 "~" H 5950 4250 50  0001 C CNN
 	1    5950 4250
@@
 F 0 "C2" V 3898 2100 50  0000 C CNN
 F 1 "100n" V 3989 2100 50  0000 C CNN
-F 2 "" H 4188 1950 50  0001 C CNN
+F 2 "Capacitors_SMD:C_0603_HandSoldering" H 4188 1950 50  0001 C CNN
 F 3 "~" H 4150 2100 50  0001 C CNN
 	1    4150 2100
@@
 F 0 "U3" H 6050 6475 50  0000 C CNN
 F 1 "AQH3213" H 6050 6384 50  0000 C CNN
-F 2 "" H 6000 6050 50  0001 C CNN
+F 2 "Housings_DIP:DIP-8_W7.62mm_SMDSocket_SmallPads" H 6000 6050 50  0001 C CNN
 F 3 "https://www3.panasonic.biz/ac/e_download/control/relay/solid-state/catalog/semi_eng_aqh.pdf" H 6000 6050 50  0001 C CNN
 	1    6000 6050
@@
 F 0 "SW1" H 5850 5135 50  0000 C CNN
 F 1 "SW_Push" H 5850 5044 50  0000 C CNN
-F 2 "" H 5850 5050 50  0001 C CNN
+F 2 "Buttons_Switches_SMD:SW_SPST_B3S-1000" H 5850 5050 50  0001 C CNN
 F 3 "" H 5850 5050 50  0001 C CNN
 	1    5850 4850
@@
 F 0 "C3" V 5598 5150 50  0000 C CNN
 F 1 "100n" V 5689 5150 50  0000 C CNN
-F 2 "" H 5888 5000 50  0001 C CNN
+F 2 "Capacitors_SMD:C_0603_HandSoldering" H 5888 5000 50  0001 C CNN
 F 3 "~" H 5850 5150 50  0001 C CNN
 	1    5850 5150
@@
 P 5400 5200
 F 0 "R1" H 5470 5246 50  0000 L CNN
-F 1 "R" H 5470 5155 50  0000 L CNN
-F 2 "" V 5330 5200 50  0001 C CNN
+F 1 "220R" H 5470 5155 50  0000 L CNN
+F 2 "Resistors_SMD:R_0603_HandSoldering" V 5330 5200 50  0001 C CNN
 F 3 "~" H 5400 5200 50  0001 C CNN
 	1    5400 5200
@@
 Wire Wire Line
 	6600 6050 6800 6050
-Text GLabel 1350 1650 2    50   Output ~ 0
+Text GLabel 1350 1750 2    50   Output ~ 0
 L_OUT
-Wire Wire Line
-	1250 1650 1350 1650
 Text GLabel 2200 2550 2    50   Input ~ 0
 L_IN
@@
 L Device:Fuse F1
 U 1 1 5C31D9DC
-P 1550 2400
-F 0 "F1" H 1610 2446 50  0000 L CNN
-F 1 "1.2 A" H 1610 2355 50  0000 L CNN
-F 2 "" V 1480 2400 50  0001 C CNN
-F 3 "~" H 1550 2400 50  0001 C CNN
-	1    1550 2400
-	1    0    0    -1
-$EndComp
-Wire Wire Line
-	1550 2250 1550 1450
-Connection ~ 1550 1450
-Wire Wire Line
-	1550 1450 1650 1450
-Wire Wire Line
-	1550 2550 2200 2550
+P 2150 2400
+F 0 "F1" H 2210 2446 50  0000 L CNN
+F 1 "BK/GMD-1.2R" H 2210 2355 50  0000 L CNN
+F 2 "Fuse_Holders_and_Fuses:Fuseholder5x20_horiz_SemiClosed_Casing10x25mm" V 2080 2400 50  0001 C CNN
+F 3 "~" H 2150 2400 50  0001 C CNN
+	1    2150 2400
+	1    0    0    -1
+$EndComp
+Wire Wire Line
+	2150 2550 2200 2550
 Wire Wire Line
 	5100 3450 5100 3550
@@
 Connection ~ 3900 2850
 Connection ~ 3350 2850
+$Comp
+L Connector:Screw_Terminal_01x04 J1
+U 1 1 5C55D2D8
+P 1050 1550
+F 0 "J1" H 970 1867 50  0000 C CNN
+F 1 "Screw_Terminal_01x04" H 970 1776 50  0000 C CNN
+F 2 "Connectors_Terminal_Blocks:TerminalBlock_bornier-4_P5.08mm" H 1050 1550 50  0001 C CNN
+F 3 "~" H 1050 1550 50  0001 C CNN
+	1    1050 1550
+	-1   0    0    -1
+$EndComp
+Wire Wire Line
+	1250 1750 1350 1750
+Wire Wire Line
+	1250 1650 1300 1650
+Wire Wire Line
+	1300 1650 1300 1550
+Connection ~ 1300 1550
+Wire Wire Line
+	1300 1550 1800 1550
+Wire Wire Line
+	1250 1450 2100 1450
+Wire Wire Line
+	2150 2250 2150 1450
+Connection ~ 2150 1450
+Wire Wire Line
+	2150 1450 2550 1450
 $EndSCHEMATC

Commit message: Fix Shematic and PCB
Parts:
- removed C4, C5: 100n, Capacitors_SMD:C_0603_HandSoldering, symbol Device:C
- added C4: 100n, Capacitors_SMD:C_0603_HandSoldering, symbol Device:C_Small
- F1: footprint Fuse_Holders_and_Fuses:Fuseholder5x20_horiz_SemiClosed_Casing10x25mm -> Fuse_Holders_and_Fuses:Fuseholder5x20_horiz_open_universal_Type-III
- J3: footprint Pin_Headers:Pin_Header_Straight_2x03_Pitch2.54mm -> Pin_Headers:Pin_Header_Straight_2x03_Pitch2.54mm_SMD
- SW1: footprint Buttons_Switches_SMD:SW_SPST_B3S-1000 -> Buttons_Switches_SMD:SW_SPST_EVQPE1
Connections:
- net GND: now also Y1.2
- net at R2.2, U2.29 (~RESET~/PC6): now also J3.5 (~RST), C4.2
- net at U2.30 (PD0): now also J2.3 (Pin_3); no longer J2.2 (Pin_2)
- net at U2.31 (PD1): now also J2.2 (Pin_2); no longer J2.3 (Pin_3)
- net at J2.1 (Pin_1): now also C4.1
Other:
- moved on the sheet: R2
Changed lines of the file:
@@
 Title "Wall-Switch Circurit"
 Date "2019-01-02"
-Rev "1"
+Rev "2"
 Comp "smart-devices.cf"
-Comment1 ""
+Comment1 "RX <> TX, Res Gnd, DTR Cap"
 Comment2 ""
 Comment3 ""
@@
 F 0 "J3" H 6620 3504 50  0000 R CNN
 F 1 "AVR-ISP-6" H 6620 3595 50  0000 R CNN
-F 2 "Pin_Headers:Pin_Header_Straight_2x03_Pitch2.54mm" V 6650 3550 50  0001 C CNN
+F 2 "Pin_Headers:Pin_Header_Straight_2x03_Pitch2.54mm_SMD" V 6650 3550 50  0001 C CNN
 F 3 " ~" H 5625 2950 50  0001 C CNN
 	1    6900 3500
@@
 	7600 3100 7600 3150
 Wire Wire Line
-	5800 3400 5800 4050
+	5800 3400 5800 4000
 Wire Wire Line
 	5800 4050 5100 4050
@@
 L Device:R R2
 U 1 1 5C2D942F
-P 6150 4050
-F 0 "R2" V 5943 4050 50  0000 C CNN
-F 1 "10k" V 6034 4050 50  0000 C CNN
-F 2 "Resistors_SMD:R_0603_HandSoldering" V 6080 4050 50  0001 C CNN
-F 3 "~" H 6150 4050 50  0001 C CNN
-	1    6150 4050
+P 6550 4000
+F 0 "R2" V 6343 4000 50  0000 C CNN
+F 1 "10k" V 6434 4000 50  0000 C CNN
+F 2 "Resistors_SMD:R_0603_HandSoldering" V 6480 4000 50  0001 C CNN
+F 3 "~" H 6550 4000 50  0001 C CNN
+	1    6550 4000
 	0    1    1    0
 $EndComp
@@
 	1    0    0    1
 $EndComp
-Wire Wire Line
-	7000 4000 7000 4050
-Wire Wire Line
-	6300 4050 7000 4050
-Connection ~ 7000 4050
-Wire Wire Line
-	7000 4050 7000 4100
-Wire Wire Line
-	6000 4050 5800 4050
 Connection ~ 5800 4050
-$Comp
-L Device:C C5
-U 1 1 5C2DC2FE
-P 6200 3400
-F 0 "C5" V 5948 3400 50  0000 C CNN
-F 1 "100n" V 6039 3400 50  0000 C CNN
-F 2 "Capacitors_SMD:C_0603_HandSoldering" H 6238 3250 50  0001 C CNN
-F 3 "~" H 6200 3400 50  0001 C CNN
-	1    6200 3400
-	0    1    1    0
-$EndComp
-Wire Wire Line
-	6500 3400 6350 3400
-Wire Wire Line
-	6050 3400 5800 3400
 Wire Wire Line
 	6500 3500 6450 3500
@@
 	1    0    0    -1
 $EndComp
-$Comp
-L Device:C C4
-U 1 1 5C2E1A18
-P 5950 4250
-F 0 "C4" V 5698 4250 50  0000 C CNN
-F 1 "100n" V 5789 4250 50  0000 C CNN
-F 2 "Capacitors_SMD:C_0603_HandSoldering" H 5988 4100 50  0001 C CNN
-F 3 "~" H 5950 4250 50  0001 C CNN
-	1    5950 4250
-	0    1    1    0
-$EndComp
-Wire Wire Line
-	6100 4250 6450 4250
 Wire Wire Line
 	5800 4250 5800 4050
 Wire Wire Line
-	6450 4350 5700 4350
-Wire Wire Line
-	5700 4350 5700 4250
-Wire Wire Line
 	5700 4250 5100 4250
-Wire Wire Line
-	6450 4450 5650 4450
-Wire Wire Line
-	5650 4450 5650 4350
-Wire Wire Line
-	5650 4350 5100 4350
 $Comp
 L power:GND #PWR010
@@
 F 0 "SW1" H 5850 5135 50  0000 C CNN
 F 1 "SW_Push" H 5850 5044 50  0000 C CNN
-F 2 "Buttons_Switches_SMD:SW_SPST_B3S-1000" H 5850 5050 50  0001 C CNN
+F 2 "Buttons_Switches_SMD:SW_SPST_EVQPE1" H 5850 5050 50  0001 C CNN
 F 3 "" H 5850 5050 50  0001 C CNN
 	1    5850 4850
@@
 F 0 "F1" H 2210 2446 50  0000 L CNN
 F 1 "BK/GMD-1.2R" H 2210 2355 50  0000 L CNN
-F 2 "Fuse_Holders_and_Fuses:Fuseholder5x20_horiz_SemiClosed_Casing10x25mm" V 2080 2400 50  0001 C CNN
+F 2 "Fuse_Holders_and_Fuses:Fuseholder5x20_horiz_open_universal_Type-III" V 2080 2400 50  0001 C CNN
 F 3 "~" H 2150 2400 50  0001 C CNN
 	1    2150 2400
@@
 Wire Wire Line
 	2150 1450 2550 1450
+Wire Wire Line
+	7000 3100 6000 3100
+Wire Wire Line
+	6000 3100 6000 3200
+Connection ~ 7000 3100
+Wire Wire Line
+	5700 4450 6450 4450
+Wire Wire Line
+	5700 4250 5700 4450
+Wire Wire Line
+	5100 4350 6450 4350
+Wire Wire Line
+	5800 3400 6500 3400
+$Comp
+L Device:C_Small C4
+U 1 1 5CCA652B
+P 5950 4250
+F 0 "C4" V 5721 4250 50  0000 C CNN
+F 1 "100n" V 5812 4250 50  0000 C CNN
+F 2 "Capacitors_SMD:C_0603_HandSoldering" H 5950 4250 50  0001 C CNN
+F 3 "~" H 5950 4250 50  0001 C CNN
+	1    5950 4250
+	0    1    1    0
+$EndComp
+Wire Wire Line
+	7000 4000 7000 4100
+Wire Wire Line
+	6700 4000 7000 4000
+Connection ~ 7000 4000
+Wire Wire Line
+	6400 4000 5800 4000
+Connection ~ 5800 4000
+Wire Wire Line
+	5800 4000 5800 4050
+Wire Wire Line
+	5800 4250 5850 4250
+Wire Wire Line
+	6050 4250 6450 4250
 $EndSCHEMATC
